Commit message: Fix Panda gripper mimic control conflict

File: src/panda_gazebo_demo/urdf/panda_hand.ros2_control.xacro (robot description, xacro)
@@ -25,5 +25,5 @@
                 </state_interface>
             </joint>
-            <joint name="panda_finger_joint2">
+            <joint name="panda_finger_joint2" mimic="false">
                 <state_interface name="position">
                     <param name="initial_value">0.0</param>
