Commit message: Add attach_and_lift_demo executable and cleanup/reset scripts for Panda robot

File: src/panda_gazebo_demo/urdf/panda.description.urdf.xacro (robot description, xacro)
@@ -275,7 +275,12 @@
         </visual>
         <collision>
-            <geometry>
-                <mesh
-                    filename="file://$(find moveit_resources_panda_description)/meshes/collision/finger.stl" />
+            <!--
+                Gazebo Bullet Featherstone assigns a 10 mm margin to the
+                default GImpact mesh path.  This primitive matches the STL
+                bounding box while preserving the original visual mesh.
+            -->
+            <origin rpy="0 0 0" xyz="0 0.013135 0.026990" />
+            <geometry>
+                <box size="0.020974 0.026536 0.053717" />
             </geometry>
         </collision>
@@ -295,8 +300,7 @@
         </visual>
         <collision>
-            <origin rpy="0 0 3.14159265359" xyz="0 0 0" />
-            <geometry>
-                <mesh
-                    filename="file://$(find moveit_resources_panda_description)/meshes/collision/finger.stl" />
+            <origin rpy="0 0 0" xyz="0 -0.013135 0.026990" />
+            <geometry>
+                <box size="0.020974 0.026536 0.053717" />
             </geometry>
         </collision>

File: src/panda_gazebo_demo/urdf/panda.gazebo.urdf.xacro (robot description, xacro)
@@ -37,4 +37,20 @@
             <parameters>$(arg controllers_file)</parameters>
         </plugin>
+        <!--
+            MoveIt's AttachedCollisionObject only changes the planning scene.
+            This Gazebo system creates the physical fixed constraint used by
+            the simulation pick / place state machine.
+        -->
+        <plugin
+            filename="gz-sim-detachable-joint-system"
+            name="gz::sim::systems::DetachableJoint">
+            <!-- panda_hand is reduced into panda_link7 by URDF-to-SDF fixed-joint lumping. -->
+            <parent_link>panda_link7</parent_link>
+            <child_model>coke</child_model>
+            <child_link>body</child_link>
+            <attach_topic>/panda/attach_coke</attach_topic>
+            <detach_topic>/panda/detach_coke</detach_topic>
+            <output_topic>/panda/coke_attached</output_topic>
+        </plugin>
     </gazebo>
 </robot>
