Commit message: Add pre-grasp planning executable and update launch files for Panda robot

File: src/panda_gazebo_demo/urdf/panda.gazebo.urdf.xacro (robot description, xacro)
@@ -8,5 +8,12 @@
         default="$(find panda_gazebo_demo)/config/controllers.yaml" />
     <!-- Import panda urdf file -->
-    <xacro:include filename="$(find moveit_resources_panda_description)/urdf/panda.urdf.xacro" />
+    <xacro:include filename="panda.description.urdf.xacro" />
+    <!-- Nominal grasp TCP at the center between the closed fingertips. -->
+    <link name="panda_tcp" />
+    <joint name="panda_tcp_joint" type="fixed">
+        <parent link="panda_hand" />
+        <child link="panda_tcp" />
+        <origin xyz="0 0 0.1034" rpy="0 0 0" />
+    </joint>
     <!-- Fix Panda base to the Gazebo world at the table-top height. -->
     <link name="world" />

Commit message: V5-T004: Panda 仿真添加 RGBD 深度相机 + ros_gz_bridge 桥接
- panda.gazebo.urdf.xacro: 新增 camera_link + 固定 joint (panda_link0→camera_link)
  位置 xyz=0.6 0 1.0, rpy=0 2.356 0 (绕Y轴135°俯视桌面)
  Gazebo rgbd_camera sensor: 640x480, 60° FOV, 10Hz
- panda_gazebo.launch.py: 新增 camera_bridge 节点
  桥接 /camera, /camera/depth, /camera/camera_info 到 ROS 2
  重映射为标准命名 /camera/color/image_raw 等

File: src/panda_gazebo_demo/urdf/panda.gazebo.urdf.xacro (robot description, xacro)
@@ -15,4 +15,22 @@
         <child link="panda_tcp" />
         <origin xyz="0 0 0.1034" rpy="0 0 0" />
+    </joint>
+    <!-- V5-T004: eye-to-hand 深度相机，固定在 panda_link0 前上方俯视桌面 -->
+    <link name="camera_link">
+        <visual>
+            <origin xyz="0 0 0" rpy="0 0 0" />
+            <geometry>
+                <box size="0.04 0.08 0.04" />
+            </geometry>
+            <material>
+                <color rgba="0.1 0.1 0.8 1.0" />
+            </material>
+        </visual>
+    </link>
+    <joint name="camera_joint" type="fixed">
+        <parent link="panda_link0" />
+        <child link="camera_link" />
+        <!-- 相机在底座前方 0.6m、高度 1.0m，绕 Y 轴转 135° 让光轴朝前下方俯视 -->
+        <origin xyz="0.6 0 1.0" rpy="0 2.356 0" />
     </joint>
     <!-- Fix Panda base to the Gazebo world at the table-top height. -->
@@ -55,3 +73,22 @@
         </plugin>
     </gazebo>
+    <!-- V5-T004: Gazebo RGBD 相机 sensor，发布 RGB + Depth + CameraInfo -->
+    <gazebo reference="camera_link">
+        <sensor name="rgbd_camera" type="rgbd_camera">
+            <topic>camera</topic>
+            <update_rate>10</update_rate>
+            <camera>
+                <horizontal_fov>1.047</horizontal_fov>
+                <image>
+                    <width>640</width>
+                    <height>480</height>
+                    <format>rgb_int8</format>
+                </image>
+                <clip>
+                    <near>0.1</near>
+                    <far>10.0</far>
+                </clip>
+            </camera>
+        </sensor>
+    </gazebo>
 </robot>

Commit message: fix: 修复 camera_link material 缺少 name 属性 + image format 改为 R8G8B8

File: src/panda_gazebo_demo/urdf/panda.gazebo.urdf.xacro (robot description, xacro)
@@ -23,5 +23,5 @@
                 <box size="0.04 0.08 0.04" />
             </geometry>
-            <material>
+            <material name="camera_blue">
                 <color rgba="0.1 0.1 0.8 1.0" />
             </material>
@@ -83,5 +83,5 @@
                     <width>640</width>
                     <height>480</height>
-                    <format>rgb_int8</format>
+                    <format>R8G8B8</format>
                 </image>
                 <clip>

Commit message: fix: 修正 camera_link RPY 为 roll=-135 pitch=0 yaw=-90
之前 rpy=0 2.356 0 导致相机X轴朝后(画面左右镜像)。
正确值 rpy=-2.356 0 -1.571 使:
- 相机Z(光轴)朝前下方 [0.707,0,-0.707]
- 相机X(画面右)朝底座-Y(右) [0,-1,0]
- 相机Y(画面下)朝后下方 [-0.707,0,-0.707]

File: src/panda_gazebo_demo/urdf/panda.gazebo.urdf.xacro (robot description, xacro)
@@ -32,5 +32,5 @@
         <child link="camera_link" />
         <!-- 相机在底座前方 0.6m、高度 1.0m，绕 Y 轴转 135° 让光轴朝前下方俯视 -->
-        <origin xyz="0.6 0 1.0" rpy="0 2.356 0" />
+        <origin xyz="0.6 0 1.0" rpy="-2.356 0 -1.571" />
     </joint>
     <!-- Fix Panda base to the Gazebo world at the table-top height. -->

Commit message: fix: 修正 SDF camera 和 URDF camera_link 的 RPY
根因: SDF camera sensor 默认光轴朝 +X, 需要绕 Y 轴转 102° 朝后下方对准桌面。
之前用的 (-2.356, 0, -1.571) 是给 URDF ROS 相机坐标系(Z朝前)算的,
在 SDF 里 camera 朝向错误, 拍不到任何物体(全灰)。

修复:
- SDF camera model pose: RPY 改为 (0, 1.782, 0)
- URDF camera_link origin: RPY 改为 (0, 1.782, 0) 保持一致
- identity TF (rgbd_camera/link/camera -> camera_link) 现在是真正的 identity

File: src/panda_gazebo_demo/urdf/panda.gazebo.urdf.xacro (robot description, xacro)
@@ -31,6 +31,6 @@
         <parent link="panda_link0" />
         <child link="camera_link" />
-        <!-- 相机在底座前方 0.6m、高度 1.0m，绕 Y 轴转 135° 让光轴朝前下方俯视 -->
-        <origin xyz="0.6 0 1.0" rpy="-2.356 0 -1.571" />
+        <!-- 相机在底座前方 0.6m、高度 1.0m，RPY 与 SDF camera model 一致 -->
+        <origin xyz="0.6 0 1.0" rpy="0 1.782 0" />
     </joint>
     <!-- Fix Panda base to the Gazebo world at the table-top height. -->

Commit message: fix: URDF camera_link RPY 改为 (0, 3.351, 0) 让 Z 朝后下方 + 去掉 identity TF
URDF camera_link (ROS相机约定 Z=光轴) 需要跟 SDF camera (默认光轴+X) 朝向一致。
SDF camera RPY (0,1.782,0) 让 +X 朝后下方。
URDF 需要 RPY (0,3.351,0) 让 +Z 朝后下方。
去掉 identity TF，感知节点直接用 camera_link 做 tf2 转换。

File: src/panda_gazebo_demo/urdf/panda.gazebo.urdf.xacro (robot description, xacro)
@@ -32,5 +32,5 @@
         <child link="camera_link" />
         <!-- 相机在底座前方 0.6m、高度 1.0m，RPY 与 SDF camera model 一致 -->
-        <origin xyz="0.6 0 1.0" rpy="0 1.782 0" />
+        <origin xyz="0.6 0 1.0" rpy="0 3.351 0" />
     </joint>
     <!-- Fix Panda base to the Gazebo world at the table-top height. -->

Commit message: fix: 相机移到侧面 (0.4,0.5,1.4) 避免机械臂挡住可乐

File: src/panda_gazebo_demo/urdf/panda.gazebo.urdf.xacro (robot description, xacro)
@@ -31,6 +31,6 @@
         <parent link="panda_link0" />
         <child link="camera_link" />
-        <!-- 相机在底座前方 0.6m、高度 1.0m，RPY 与 SDF camera model 一致 -->
-        <origin xyz="0.6 0 1.0" rpy="0 3.351 0" />
+        <!-- 相机在底座侧前方 0.4m/Y0.5m、高度 0.625m(相对link0)，避免机械臂挡住视线 -->
+        <origin xyz="0.4 0.5 0.625" rpy="0 2.4065 -1.7682" />
     </joint>
     <!-- Fix Panda base to the Gazebo world at the table-top height. -->
