Commit message: feat: establish SO-101 simulation observation prerequisites

File: src/so101_gazebo_demo/urdf/so101_base.xacro (robot description, xacro)
@@ -6,4 +6,6 @@
 -->
 <robot xmlns:xacro="http://www.ros.org/wiki/xacro">
+	<!-- Keep MoveIt on the detailed meshes; Gazebo opts into contact pads. -->
+	<xacro:arg name="gazebo_collision_primitives" default="false" />
 	<!-- Links -->
 	<link name="world" />
@@ -291,10 +293,12 @@
 			<material name="sts3215" />
 		</visual>
-		<collision>
-			<origin xyz="0.0077 0.0001 -0.0234" rpy="-1.5708 -5.55112e-17 -1.38213e-14" />
-			<geometry>
-				<mesh filename="package://so101_gazebo_demo/meshes/so101/sts3215_03a_v1.stl" />
-			</geometry>
-		</collision>
+		<xacro:unless value="$(arg gazebo_collision_primitives)">
+			<collision>
+				<origin xyz="0.0077 0.0001 -0.0234" rpy="-1.5708 -5.55112e-17 -1.38213e-14" />
+				<geometry>
+					<mesh filename="package://so101_gazebo_demo/meshes/so101/sts3215_03a_v1.stl" />
+				</geometry>
+			</collision>
+		</xacro:unless>
 		<!-- Part wrist_roll_follower_so101_v1 -->
 		<visual>
@@ -307,12 +311,23 @@
 			<material name="3d_printed" />
 		</visual>
-		<collision>
-			<origin xyz="5.55112e-17 -0.000218214 0.000949706"
-				rpy="-3.14159 -5.55112e-17 -9.17912e-24" />
-			<geometry>
-				<mesh
-					filename="package://so101_gazebo_demo/meshes/so101/wrist_roll_follower_so101_v1.stl" />
-			</geometry>
-		</collision>
+		<xacro:unless value="$(arg gazebo_collision_primitives)">
+			<collision>
+				<origin xyz="5.55112e-17 -0.000218214 0.000949706"
+					rpy="-3.14159 -5.55112e-17 -9.17912e-24" />
+				<geometry>
+					<mesh
+						filename="package://so101_gazebo_demo/meshes/so101/wrist_roll_follower_so101_v1.stl" />
+				</geometry>
+			</collision>
+		</xacro:unless>
+		<xacro:if value="$(arg gazebo_collision_primitives)">
+			<!-- Convex fingertip pad used for load-bearing Coke contact in DART. -->
+			<collision name="fixed_finger_contact">
+				<origin xyz="-0.004 0 -0.084" rpy="0 0 0" />
+				<geometry>
+					<box size="0.016 0.020 0.042" />
+				</geometry>
+			</collision>
+		</xacro:if>
 	</link>
 	<!-- Link jaw -->
@@ -332,10 +347,21 @@
 			<material name="3d_printed" />
 		</visual>
-		<collision>
-			<origin xyz="-5.55112e-17 -1.94746e-17 0.0189" rpy="9.53145e-17 -4.66093e-24 0" />
-			<geometry>
-				<mesh filename="package://so101_gazebo_demo/meshes/so101/moving_jaw_so101_v1.stl" />
-			</geometry>
-		</collision>
+		<xacro:unless value="$(arg gazebo_collision_primitives)">
+			<collision>
+				<origin xyz="-5.55112e-17 -1.94746e-17 0.0189" rpy="9.53145e-17 -4.66093e-24 0" />
+				<geometry>
+					<mesh filename="package://so101_gazebo_demo/meshes/so101/moving_jaw_so101_v1.stl" />
+				</geometry>
+			</collision>
+		</xacro:unless>
+		<xacro:if value="$(arg gazebo_collision_primitives)">
+			<!-- Moving fingertip pad follows joint 6 and supports Coke contact. -->
+			<collision name="moving_finger_contact">
+				<origin xyz="-0.009 -0.070 0" rpy="0 0 0" />
+				<geometry>
+					<box size="0.010 0.026 0.028" />
+				</geometry>
+			</collision>
+		</xacro:if>
 	</link>
 	<!-- Joint from gripper to jaw -->

File: src/so101_gazebo_demo/urdf/so101_gazebo.xacro (robot description, xacro)
@@ -6,4 +6,20 @@
             <parameters>$(find so101_gazebo_demo)/config/so101_controllers.yaml</parameters>
         </plugin>
+        <!--
+          This must name a link entity that survives URDF-to-SDF conversion.
+          The running Gazebo scene graph exposes gripper directly under so101.
+          The output is an edge-triggered event; a later relay owns durable state.
+        -->
+        <plugin
+            filename="gz-sim-detachable-joint-system"
+            name="gz::sim::systems::DetachableJoint">
+            <parent_link>gripper</parent_link>
+            <child_model>coke</child_model>
+            <child_link>body</child_link>
+            <initially_detached>true</initially_detached>
+            <attach_topic>/so101/attach_coke</attach_topic>
+            <detach_topic>/so101/detach_coke</detach_topic>
+            <output_topic>/so101/coke_attached_event</output_topic>
+        </plugin>
     </gazebo>
 </robot>

File: src/so101_gazebo_demo/urdf/so101_ros2_control.xacro (robot description, xacro)
@@ -12,4 +12,5 @@
             </command_interface>
             <state_interface name="position" />
+            <state_interface name="velocity" />
         </joint>
         <joint name="2">
@@ -19,4 +20,5 @@
             </command_interface>
             <state_interface name="position" />
+            <state_interface name="velocity" />
         </joint>
         <joint name="3">
@@ -26,4 +28,5 @@
             </command_interface>
             <state_interface name="position" />
+            <state_interface name="velocity" />
         </joint>
         <joint name="4">
@@ -33,4 +36,5 @@
             </command_interface>
             <state_interface name="position" />
+            <state_interface name="velocity" />
         </joint>
         <joint name="5">
@@ -40,4 +44,5 @@
             </command_interface>
             <state_interface name="position" />
+            <state_interface name="velocity" />
         </joint>
         <joint name="6">
@@ -47,4 +52,5 @@
             </command_interface>
             <state_interface name="position" />
+            <state_interface name="velocity" />
         </joint>
     </ros2_control>

Commit message: fix(so101): validate simulated grasp through lift

File: src/so101_gazebo_demo/urdf/so101_base.xacro (robot description, xacro)
@@ -322,7 +322,9 @@
 		</xacro:unless>
 		<xacro:if value="$(arg gazebo_collision_primitives)">
-			<!-- Convex fingertip pad used for load-bearing Coke contact in DART. -->
+			<!-- Convex fingertip pad used for load-bearing Coke contact in DART.
+			     Keep 2 mm pre-open clearance from the nominal Coke surface: an
+			     exactly tangent rigid-body start is unstable in the simulator. -->
 			<collision name="fixed_finger_contact">
-				<origin xyz="-0.004 0 -0.084" rpy="0 0 0" />
+				<origin xyz="-0.0216 0 -0.084" rpy="0 0 0" />
 				<geometry>
 					<box size="0.016 0.020 0.042" />
@@ -358,5 +360,5 @@
 			<!-- Moving fingertip pad follows joint 6 and supports Coke contact. -->
 			<collision name="moving_finger_contact">
-				<origin xyz="-0.009 -0.070 0" rpy="0 0 0" />
+				<origin xyz="-0.01599174 -0.09546963 0" rpy="0 0 0" />
 				<geometry>
 					<box size="0.010 0.026 0.028" />

Commit message: Refine SO-101 gripper simulation and debug tooling

File: src/so101_gazebo_demo/urdf/so101_base.xacro (robot description, xacro)
@@ -8,4 +8,13 @@
 	<!-- Keep MoveIt on the detailed meshes; Gazebo opts into contact pads. -->
 	<xacro:arg name="gazebo_collision_primitives" default="false" />
+	<xacro:macro name="moving_jaw_convex_collision" params="piece">
+		<collision name="${piece}">
+			<origin xyz="-5.55112e-17 -1.94746e-17 0.0189"
+				rpy="9.53145e-17 -4.66093e-24 0" />
+			<geometry>
+				<mesh filename="package://so101_gazebo_demo/meshes/so101/collision/${piece}.stl" />
+			</geometry>
+		</collision>
+	</xacro:macro>
 	<!-- Links -->
 	<link name="world" />
@@ -358,11 +367,69 @@
 		</xacro:unless>
 		<xacro:if value="$(arg gazebo_collision_primitives)">
-			<!-- Moving fingertip pad follows joint 6 and supports Coke contact. -->
-			<collision name="moving_finger_contact">
-				<origin xyz="-0.01599174 -0.09546963 0" rpy="0 0 0" />
-				<geometry>
-					<box size="0.010 0.026 0.028" />
-				</geometry>
-			</collision>
+			<!-- Offline VHACD pieces keep the long jaw's interior concavity open. -->
+			<xacro:moving_jaw_convex_collision piece="moving_jaw_convex_000" />
+			<xacro:moving_jaw_convex_collision piece="moving_jaw_convex_001" />
+			<xacro:moving_jaw_convex_collision piece="moving_jaw_convex_002" />
+			<xacro:moving_jaw_convex_collision piece="moving_jaw_convex_003" />
+			<xacro:moving_jaw_convex_collision piece="moving_jaw_convex_004" />
+			<xacro:moving_jaw_convex_collision piece="moving_jaw_convex_005" />
+			<xacro:moving_jaw_convex_collision piece="moving_jaw_convex_006" />
+			<xacro:moving_jaw_convex_collision piece="moving_jaw_convex_007" />
+			<xacro:moving_jaw_convex_collision piece="moving_jaw_convex_008" />
+			<xacro:moving_jaw_convex_collision piece="moving_jaw_convex_009" />
+			<xacro:moving_jaw_convex_collision piece="moving_jaw_convex_010" />
+			<xacro:moving_jaw_convex_collision piece="moving_jaw_convex_011" />
+			<xacro:moving_jaw_convex_collision piece="moving_jaw_convex_012" />
+			<xacro:moving_jaw_convex_collision piece="moving_jaw_convex_013" />
+			<xacro:moving_jaw_convex_collision piece="moving_jaw_convex_014" />
+			<xacro:moving_jaw_convex_collision piece="moving_jaw_convex_015" />
+			<xacro:moving_jaw_convex_collision piece="moving_jaw_convex_016" />
+			<xacro:moving_jaw_convex_collision piece="moving_jaw_convex_017" />
+			<xacro:moving_jaw_convex_collision piece="moving_jaw_convex_018" />
+			<xacro:moving_jaw_convex_collision piece="moving_jaw_convex_019" />
+			<xacro:moving_jaw_convex_collision piece="moving_jaw_convex_020" />
+			<xacro:moving_jaw_convex_collision piece="moving_jaw_convex_021" />
+			<xacro:moving_jaw_convex_collision piece="moving_jaw_convex_022" />
+			<xacro:moving_jaw_convex_collision piece="moving_jaw_convex_023" />
+			<xacro:moving_jaw_convex_collision piece="moving_jaw_convex_024" />
+			<xacro:moving_jaw_convex_collision piece="moving_jaw_convex_025" />
+			<xacro:moving_jaw_convex_collision piece="moving_jaw_convex_026" />
+			<xacro:moving_jaw_convex_collision piece="moving_jaw_convex_027" />
+			<xacro:moving_jaw_convex_collision piece="moving_jaw_convex_028" />
+			<xacro:moving_jaw_convex_collision piece="moving_jaw_convex_029" />
+			<xacro:moving_jaw_convex_collision piece="moving_jaw_convex_030" />
+			<xacro:moving_jaw_convex_collision piece="moving_jaw_convex_031" />
+			<xacro:moving_jaw_convex_collision piece="moving_jaw_convex_032" />
+			<xacro:moving_jaw_convex_collision piece="moving_jaw_convex_033" />
+			<xacro:moving_jaw_convex_collision piece="moving_jaw_convex_034" />
+			<xacro:moving_jaw_convex_collision piece="moving_jaw_convex_035" />
+			<xacro:moving_jaw_convex_collision piece="moving_jaw_convex_036" />
+			<xacro:moving_jaw_convex_collision piece="moving_jaw_convex_037" />
+			<xacro:moving_jaw_convex_collision piece="moving_jaw_convex_038" />
+			<xacro:moving_jaw_convex_collision piece="moving_jaw_convex_039" />
+			<xacro:moving_jaw_convex_collision piece="moving_jaw_convex_040" />
+			<xacro:moving_jaw_convex_collision piece="moving_jaw_convex_041" />
+			<xacro:moving_jaw_convex_collision piece="moving_jaw_convex_042" />
+			<xacro:moving_jaw_convex_collision piece="moving_jaw_convex_043" />
+			<xacro:moving_jaw_convex_collision piece="moving_jaw_convex_044" />
+			<xacro:moving_jaw_convex_collision piece="moving_jaw_convex_045" />
+			<xacro:moving_jaw_convex_collision piece="moving_jaw_convex_046" />
+			<xacro:moving_jaw_convex_collision piece="moving_jaw_convex_047" />
+			<xacro:moving_jaw_convex_collision piece="moving_jaw_convex_048" />
+			<xacro:moving_jaw_convex_collision piece="moving_jaw_convex_049" />
+			<xacro:moving_jaw_convex_collision piece="moving_jaw_convex_050" />
+			<xacro:moving_jaw_convex_collision piece="moving_jaw_convex_051" />
+			<xacro:moving_jaw_convex_collision piece="moving_jaw_convex_052" />
+			<xacro:moving_jaw_convex_collision piece="moving_jaw_convex_053" />
+			<xacro:moving_jaw_convex_collision piece="moving_jaw_convex_054" />
+			<xacro:moving_jaw_convex_collision piece="moving_jaw_convex_055" />
+			<xacro:moving_jaw_convex_collision piece="moving_jaw_convex_056" />
+			<xacro:moving_jaw_convex_collision piece="moving_jaw_convex_057" />
+			<xacro:moving_jaw_convex_collision piece="moving_jaw_convex_058" />
+			<xacro:moving_jaw_convex_collision piece="moving_jaw_convex_059" />
+			<xacro:moving_jaw_convex_collision piece="moving_jaw_convex_060" />
+			<xacro:moving_jaw_convex_collision piece="moving_jaw_convex_061" />
+			<xacro:moving_jaw_convex_collision piece="moving_jaw_convex_062" />
+			<xacro:moving_jaw_convex_collision piece="moving_jaw_convex_063" />
 		</xacro:if>
 	</link>
