Commit message: feat(so101): add simulation teleop and harden physical pick-place validation
Configure the light cup world, calibrated motion targets, controller limits, and validation policies.

Add TPU fingertip geometry, generated VHACD contact collision meshes, gap calibration, and deterministic asset tooling.

Harden physical grasp validation, micro-lift evidence, state-machine stepping, checkpoints, recovery, and the bounded force-continue path.

Coordinate Gazebo and MoveIt attach/detach, planning-scene initialization and observation, reset ownership, readiness, scene revision, and simulation-session invalidation.

Add the simulation-only FastAPI Teleop server and React/Vite/shadcn Web UI with expanded Tailwind/PostCSS production styling.

Expose live joint, TCP, object pose, contact, collision, attachment, controller, and source-age telemetry.

Render structured collision and contact evidence in stable shadcn panels, add accessible top-level Tabs and TCP ButtonGroup controls, and keep connection actions stable as live metadata changes.

Preflight the production Web bundle during one-command launch, use Bun with its authoritative lockfile, rebuild missing or stale assets, and fail closed before FastAPI on build errors.

Apply a uniform two-degree joint safety margin, distinguish arm and gripper execution, wait up to one minute for TCP IK, and expose backend error codes through global toasts.

Support Plan, Execute, Home, Reset, screenshots, parameter save/load, workflow pause/resume/step, and auditable command leases.

Add recording and video diagnostic helpers plus Gazebo camera, maximize, tiling, and startup troubleshooting support.

Document the design and Chinese operator workflow, expand C++/Python/Bun/Playwright tests, and ignore Python, Node, Playwright, and generated workspace artifacts.

File: src/so101_gazebo_demo/urdf/so101_base.xacro (robot description, xacro)
@@ -8,12 +8,54 @@
 	<!-- Keep MoveIt on the detailed meshes; Gazebo opts into contact pads. -->
 	<xacro:arg name="gazebo_collision_primitives" default="false" />
-	<xacro:macro name="moving_jaw_convex_collision" params="piece">
+	<xacro:arg name="object_config" default="" />
+	<xacro:macro name="fingertip_convex_collision" params="piece directory xyz rpy">
 		<collision name="${piece}">
-			<origin xyz="-5.55112e-17 -1.94746e-17 0.0189"
-				rpy="9.53145e-17 -4.66093e-24 0" />
-			<geometry>
-				<mesh filename="package://so101_gazebo_demo/meshes/so101/collision/${piece}.stl" />
-			</geometry>
-		</collision>
+			<origin xyz="${xyz}" rpy="${rpy}" />
+			<geometry>
+				<mesh filename="package://so101_gazebo_demo/meshes/so101/collision/${directory}/${piece}.stl" />
+			</geometry>
+		</collision>
+	</xacro:macro>
+	<xacro:macro name="fingertip_pad_visual" params="name xyz rpy mesh">
+		<visual name="${name}_visual">
+			<origin xyz="${xyz}" rpy="${rpy}" />
+			<geometry><mesh filename="${mesh}" /></geometry>
+			<material name="tpu_95a_adapter" />
+		</visual>
+	</xacro:macro>
+	<xacro:macro name="fingertip_pad_collision" params="name xyz rpy mesh">
+		<collision name="${name}">
+			<origin xyz="${xyz}" rpy="${rpy}" />
+			<geometry><mesh filename="${mesh}" /></geometry>
+		</collision>
+	</xacro:macro>
+	<xacro:macro name="configured_fixed_fingertip_pad" params="xyz rpy">
+		<xacro:if value="${'$(arg object_config)' != ''}">
+			<xacro:property name="pads" value="${xacro.load_yaml('$(arg object_config)')['fingertip_pads']}" />
+			<xacro:if value="${pads['enabled']}">
+				<xacro:fingertip_pad_visual name="fixed_fingertip_pad" xyz="${xyz}" rpy="${rpy}" mesh="package://so101_gazebo_demo/meshes/so101/generated/fixed/fingertip_pad.stl" />
+				<xacro:fingertip_pad_collision name="fixed_fingertip_pad_collision_000" xyz="${xyz}" rpy="${rpy}" mesh="package://so101_gazebo_demo/meshes/so101/generated/fixed/fingertip_pad_collision_000.stl" />
+				<xacro:fingertip_pad_collision name="fixed_fingertip_pad_collision_001" xyz="${xyz}" rpy="${rpy}" mesh="package://so101_gazebo_demo/meshes/so101/generated/fixed/fingertip_pad_collision_001.stl" />
+				<xacro:fingertip_pad_collision name="fixed_fingertip_pad_collision_002" xyz="${xyz}" rpy="${rpy}" mesh="package://so101_gazebo_demo/meshes/so101/generated/fixed/fingertip_pad_collision_002.stl" />
+				<xacro:fingertip_pad_collision name="fixed_fingertip_pad_collision_003" xyz="${xyz}" rpy="${rpy}" mesh="package://so101_gazebo_demo/meshes/so101/generated/fixed/fingertip_pad_collision_003.stl" />
+				<xacro:fingertip_pad_collision name="fixed_fingertip_pad_collision_004" xyz="${xyz}" rpy="${rpy}" mesh="package://so101_gazebo_demo/meshes/so101/generated/fixed/fingertip_pad_collision_004.stl" />
+				<xacro:fingertip_pad_collision name="fixed_fingertip_pad_collision_005" xyz="${xyz}" rpy="${rpy}" mesh="package://so101_gazebo_demo/meshes/so101/generated/fixed/fingertip_pad_collision_005.stl" />
+				<xacro:fingertip_pad_collision name="fixed_fingertip_pad_collision_006" xyz="${xyz}" rpy="${rpy}" mesh="package://so101_gazebo_demo/meshes/so101/generated/fixed/fingertip_pad_collision_006.stl" />
+			</xacro:if>
+		</xacro:if>
+	</xacro:macro>
+	<xacro:macro name="configured_moving_fingertip_pad" params="xyz rpy">
+		<xacro:if value="${'$(arg object_config)' != ''}">
+			<xacro:property name="pads" value="${xacro.load_yaml('$(arg object_config)')['fingertip_pads']}" />
+			<xacro:if value="${pads['enabled']}">
+				<xacro:fingertip_pad_visual name="moving_fingertip_pad" xyz="${xyz}" rpy="${rpy}" mesh="package://so101_gazebo_demo/meshes/so101/generated/moving/fingertip_pad.stl" />
+				<xacro:fingertip_pad_collision name="moving_fingertip_pad_collision_000" xyz="${xyz}" rpy="${rpy}" mesh="package://so101_gazebo_demo/meshes/so101/generated/moving/fingertip_pad_collision_000.stl" />
+				<xacro:fingertip_pad_collision name="moving_fingertip_pad_collision_001" xyz="${xyz}" rpy="${rpy}" mesh="package://so101_gazebo_demo/meshes/so101/generated/moving/fingertip_pad_collision_001.stl" />
+				<xacro:fingertip_pad_collision name="moving_fingertip_pad_collision_002" xyz="${xyz}" rpy="${rpy}" mesh="package://so101_gazebo_demo/meshes/so101/generated/moving/fingertip_pad_collision_002.stl" />
+				<xacro:fingertip_pad_collision name="moving_fingertip_pad_collision_003" xyz="${xyz}" rpy="${rpy}" mesh="package://so101_gazebo_demo/meshes/so101/generated/moving/fingertip_pad_collision_003.stl" />
+				<xacro:fingertip_pad_collision name="moving_fingertip_pad_collision_004" xyz="${xyz}" rpy="${rpy}" mesh="package://so101_gazebo_demo/meshes/so101/generated/moving/fingertip_pad_collision_004.stl" />
+				<xacro:fingertip_pad_collision name="moving_fingertip_pad_collision_005" xyz="${xyz}" rpy="${rpy}" mesh="package://so101_gazebo_demo/meshes/so101/generated/moving/fingertip_pad_collision_005.stl" />
+			</xacro:if>
+		</xacro:if>
 	</xacro:macro>
 	<!-- Links -->
@@ -30,4 +72,8 @@
 	<material name="sts3215">
 		<color rgba="0.1 0.1 0.1 1.0" />
+	</material>
+	<!-- TPU 95A semantic; Gazebo still uses rigid primitive contact geometry. -->
+	<material name="tpu_95a_adapter">
+		<color rgba="0.10 0.45 0.95 1.0" />
 	</material>
 	<!-- Link base -->
@@ -331,14 +377,14 @@
 		</xacro:unless>
 		<xacro:if value="$(arg gazebo_collision_primitives)">
-			<!-- Convex fingertip pad used for load-bearing Coke contact in DART.
-			     Keep 2 mm pre-open clearance from the nominal Coke surface: an
-			     exactly tangent rigid-body start is unstable in the simulator. -->
-			<collision name="fixed_finger_contact">
-				<origin xyz="-0.0216 0 -0.084" rpy="0 0 0" />
-				<geometry>
-					<box size="0.016 0.020 0.042" />
-				</geometry>
-			</collision>
+			<!-- Offline VHACD for the load-bearing fixed fingertip only. -->
+			<xacro:fingertip_convex_collision piece="fixed_finger_contact_convex_000" directory="fixed_finger_contact" xyz="5.55112e-17 -0.000218214 0.000949706" rpy="-3.14159 -5.55112e-17 -9.17912e-24" />
+			<xacro:fingertip_convex_collision piece="fixed_finger_contact_convex_001" directory="fixed_finger_contact" xyz="5.55112e-17 -0.000218214 0.000949706" rpy="-3.14159 -5.55112e-17 -9.17912e-24" />
+			<xacro:fingertip_convex_collision piece="fixed_finger_contact_convex_002" directory="fixed_finger_contact" xyz="5.55112e-17 -0.000218214 0.000949706" rpy="-3.14159 -5.55112e-17 -9.17912e-24" />
+			<xacro:fingertip_convex_collision piece="fixed_finger_contact_convex_003" directory="fixed_finger_contact" xyz="5.55112e-17 -0.000218214 0.000949706" rpy="-3.14159 -5.55112e-17 -9.17912e-24" />
+			<xacro:fingertip_convex_collision piece="fixed_finger_contact_convex_004" directory="fixed_finger_contact" xyz="5.55112e-17 -0.000218214 0.000949706" rpy="-3.14159 -5.55112e-17 -9.17912e-24" />
+			<xacro:fingertip_convex_collision piece="fixed_finger_contact_convex_005" directory="fixed_finger_contact" xyz="5.55112e-17 -0.000218214 0.000949706" rpy="-3.14159 -5.55112e-17 -9.17912e-24" />
+			<xacro:fingertip_convex_collision piece="fixed_finger_contact_convex_006" directory="fixed_finger_contact" xyz="5.55112e-17 -0.000218214 0.000949706" rpy="-3.14159 -5.55112e-17 -9.17912e-24" />
 		</xacro:if>
+		<xacro:configured_fixed_fingertip_pad xyz="5.55112e-17 -0.000218214 0.000949706" rpy="-3.14159 -5.55112e-17 -9.17912e-24" />
 	</link>
 	<!-- Link jaw -->
@@ -367,70 +413,15 @@
 		</xacro:unless>
 		<xacro:if value="$(arg gazebo_collision_primitives)">
-			<!-- Offline VHACD pieces keep the long jaw's interior concavity open. -->
-			<xacro:moving_jaw_convex_collision piece="moving_jaw_convex_000" />
-			<xacro:moving_jaw_convex_collision piece="moving_jaw_convex_001" />
-			<xacro:moving_jaw_convex_collision piece="moving_jaw_convex_002" />
-			<xacro:moving_jaw_convex_collision piece="moving_jaw_convex_003" />
-			<xacro:moving_jaw_convex_collision piece="moving_jaw_convex_004" />
-			<xacro:moving_jaw_convex_collision piece="moving_jaw_convex_005" />
-			<xacro:moving_jaw_convex_collision piece="moving_jaw_convex_006" />
-			<xacro:moving_jaw_convex_collision piece="moving_jaw_convex_007" />
-			<xacro:moving_jaw_convex_collision piece="moving_jaw_convex_008" />
-			<xacro:moving_jaw_convex_collision piece="moving_jaw_convex_009" />
-			<xacro:moving_jaw_convex_collision piece="moving_jaw_convex_010" />
-			<xacro:moving_jaw_convex_collision piece="moving_jaw_convex_011" />
-			<xacro:moving_jaw_convex_collision piece="moving_jaw_convex_012" />
-			<xacro:moving_jaw_convex_collision piece="moving_jaw_convex_013" />
-			<xacro:moving_jaw_convex_collision piece="moving_jaw_convex_014" />
-			<xacro:moving_jaw_convex_collision piece="moving_jaw_convex_015" />
-			<xacro:moving_jaw_convex_collision piece="moving_jaw_convex_016" />
-			<xacro:moving_jaw_convex_collision piece="moving_jaw_convex_017" />
-			<xacro:moving_jaw_convex_collision piece="moving_jaw_convex_018" />
-			<xacro:moving_jaw_convex_collision piece="moving_jaw_convex_019" />
-			<xacro:moving_jaw_convex_collision piece="moving_jaw_convex_020" />
-			<xacro:moving_jaw_convex_collision piece="moving_jaw_convex_021" />
-			<xacro:moving_jaw_convex_collision piece="moving_jaw_convex_022" />
-			<xacro:moving_jaw_convex_collision piece="moving_jaw_convex_023" />
-			<xacro:moving_jaw_convex_collision piece="moving_jaw_convex_024" />
-			<xacro:moving_jaw_convex_collision piece="moving_jaw_convex_025" />
-			<xacro:moving_jaw_convex_collision piece="moving_jaw_convex_026" />
-			<xacro:moving_jaw_convex_collision piece="moving_jaw_convex_027" />
-			<xacro:moving_jaw_convex_collision piece="moving_jaw_convex_028" />
-			<xacro:moving_jaw_convex_collision piece="moving_jaw_convex_029" />
-			<xacro:moving_jaw_convex_collision piece="moving_jaw_convex_030" />
-			<xacro:moving_jaw_convex_collision piece="moving_jaw_convex_031" />
-			<xacro:moving_jaw_convex_collision piece="moving_jaw_convex_032" />
-			<xacro:moving_jaw_convex_collision piece="moving_jaw_convex_033" />
-			<xacro:moving_jaw_convex_collision piece="moving_jaw_convex_034" />
-			<xacro:moving_jaw_convex_collision piece="moving_jaw_convex_035" />
-			<xacro:moving_jaw_convex_collision piece="moving_jaw_convex_036" />
-			<xacro:moving_jaw_convex_collision piece="moving_jaw_convex_037" />
-			<xacro:moving_jaw_convex_collision piece="moving_jaw_convex_038" />
-			<xacro:moving_jaw_convex_collision piece="moving_jaw_convex_039" />
-			<xacro:moving_jaw_convex_collision piece="moving_jaw_convex_040" />
-			<xacro:moving_jaw_convex_collision piece="moving_jaw_convex_041" />
-			<xacro:moving_jaw_convex_collision piece="moving_jaw_convex_042" />
-			<xacro:moving_jaw_convex_collision piece="moving_jaw_convex_043" />
-			<xacro:moving_jaw_convex_collision piece="moving_jaw_convex_044" />
-			<xacro:moving_jaw_convex_collision piece="moving_jaw_convex_045" />
-			<xacro:moving_jaw_convex_collision piece="moving_jaw_convex_046" />
-			<xacro:moving_jaw_convex_collision piece="moving_jaw_convex_047" />
-			<xacro:moving_jaw_convex_collision piece="moving_jaw_convex_048" />
-			<xacro:moving_jaw_convex_collision piece="moving_jaw_convex_049" />
-			<xacro:moving_jaw_convex_collision piece="moving_jaw_convex_050" />
-			<xacro:moving_jaw_convex_collision piece="moving_jaw_convex_051" />
-			<xacro:moving_jaw_convex_collision piece="moving_jaw_convex_052" />
-			<xacro:moving_jaw_convex_collision piece="moving_jaw_convex_053" />
-			<xacro:moving_jaw_convex_collision piece="moving_jaw_convex_054" />
-			<xacro:moving_jaw_convex_collision piece="moving_jaw_convex_055" />
-			<xacro:moving_jaw_convex_collision piece="moving_jaw_convex_056" />
-			<xacro:moving_jaw_convex_collision piece="moving_jaw_convex_057" />
-			<xacro:moving_jaw_convex_collision piece="moving_jaw_convex_058" />
-			<xacro:moving_jaw_convex_collision piece="moving_jaw_convex_059" />
-			<xacro:moving_jaw_convex_collision piece="moving_jaw_convex_060" />
-			<xacro:moving_jaw_convex_collision piece="moving_jaw_convex_061" />
-			<xacro:moving_jaw_convex_collision piece="moving_jaw_convex_062" />
-			<xacro:moving_jaw_convex_collision piece="moving_jaw_convex_063" />
+			<!-- Offline VHACD for the moving load-bearing fingertip only. -->
+			<xacro:fingertip_convex_collision piece="moving_jaw_contact_convex_000" directory="moving_jaw_contact" xyz="-5.55112e-17 -1.94746e-17 0.0189" rpy="9.53145e-17 -4.66093e-24 0" />
+			<xacro:fingertip_convex_collision piece="moving_jaw_contact_convex_001" directory="moving_jaw_contact" xyz="-5.55112e-17 -1.94746e-17 0.0189" rpy="9.53145e-17 -4.66093e-24 0" />
+			<xacro:fingertip_convex_collision piece="moving_jaw_contact_convex_002" directory="moving_jaw_contact" xyz="-5.55112e-17 -1.94746e-17 0.0189" rpy="9.53145e-17 -4.66093e-24 0" />
+			<xacro:fingertip_convex_collision piece="moving_jaw_contact_convex_003" directory="moving_jaw_contact" xyz="-5.55112e-17 -1.94746e-17 0.0189" rpy="9.53145e-17 -4.66093e-24 0" />
+			<xacro:fingertip_convex_collision piece="moving_jaw_contact_convex_004" directory="moving_jaw_contact" xyz="-5.55112e-17 -1.94746e-17 0.0189" rpy="9.53145e-17 -4.66093e-24 0" />
+			<xacro:fingertip_convex_collision piece="moving_jaw_contact_convex_005" directory="moving_jaw_contact" xyz="-5.55112e-17 -1.94746e-17 0.0189" rpy="9.53145e-17 -4.66093e-24 0" />
+			<xacro:fingertip_convex_collision piece="moving_jaw_contact_convex_006" directory="moving_jaw_contact" xyz="-5.55112e-17 -1.94746e-17 0.0189" rpy="9.53145e-17 -4.66093e-24 0" />
+			<xacro:fingertip_convex_collision piece="moving_jaw_contact_convex_007" directory="moving_jaw_contact" xyz="-5.55112e-17 -1.94746e-17 0.0189" rpy="9.53145e-17 -4.66093e-24 0" />
 		</xacro:if>
+		<xacro:configured_moving_fingertip_pad xyz="-5.55112e-17 -1.94746e-17 0.0189" rpy="9.53145e-17 -4.66093e-24 0" />
 	</link>
 	<!-- Joint from gripper to jaw -->
@@ -440,5 +431,5 @@
 		<child link="jaw" />
 		<axis xyz="0 0 1" />
-		<limit effort="10" velocity="10" lower="-0.174533" upper="1.74533" />
+		<limit effort="10" velocity="10" lower="-0.059303612618397" upper="1.74533" />
 	</joint>
 	<transmission name="6_trans">

File: src/so101_gazebo_demo/urdf/so101_gazebo.xacro (robot description, xacro)
@@ -15,10 +15,25 @@
             name="gz::sim::systems::DetachableJoint">
             <parent_link>gripper</parent_link>
-            <child_model>coke</child_model>
+            <child_model>plastic_cup</child_model>
             <child_link>body</child_link>
             <initially_detached>true</initially_detached>
-            <attach_topic>/so101/attach_coke</attach_topic>
-            <detach_topic>/so101/detach_coke</detach_topic>
-            <output_topic>/so101/coke_attached_event</output_topic>
+            <attach_topic>/so101/attach_object</attach_topic>
+            <detach_topic>/so101/detach_object</detach_topic>
+            <output_topic>/so101/object_attached_event</output_topic>
+        </plugin>
+        <!--
+          Contact is physical until attach validation succeeds. During rigid
+          carry the DetachableJoint is authoritative, so disable TaskObject collision
+          response to avoid locking fingertip penetration into a constraint loop.
+          Detach re-enables collision before the TaskObject settles on the table.
+        -->
+        <plugin
+            filename="libso101_attachment_collision_system.so"
+            name="so101_gazebo_demo::AttachmentCollisionSystem">
+            <child_model>plastic_cup</child_model>
+            <attach_topic>/so101/attach_object</attach_topic>
+            <detach_topic>/so101/detach_object</detach_topic>
+            <joint_state_topic>/so101/object_attached</joint_state_topic>
+            <collision_state_topic>/so101/object_collision_enabled</collision_state_topic>
         </plugin>
     </gazebo>

File: src/so101_gazebo_demo/urdf/so101_ros2_control.xacro (robot description, xacro)
@@ -48,5 +48,5 @@
         <joint name="6">
             <command_interface name="position">
-                <param name="min">-0.174533</param>
+                <param name="min">-0.059303612618397</param>
                 <param name="max">1.74533</param>
             </command_interface>

Commit message: fix(so101): preserve friction grasp baseline

File: src/so101_gazebo_demo/urdf/so101_base.xacro (robot description, xacro)
@@ -398,5 +398,5 @@
 		<!-- Part moving_jaw_so101_v1 -->
 		<visual>
-			<origin xyz="-5.55112e-17 -1.94746e-17 0.0189" rpy="9.53145e-17 -4.66093e-24 0" />
+			<origin xyz="-5.55112e-17 0.0004 0.0189" rpy="9.53145e-17 -4.66093e-24 0" />
 			<geometry>
 				<mesh filename="package://so101_gazebo_demo/meshes/so101/moving_jaw_so101_v1.stl" />
@@ -406,5 +406,5 @@
 		<xacro:unless value="$(arg gazebo_collision_primitives)">
 			<collision>
-				<origin xyz="-5.55112e-17 -1.94746e-17 0.0189" rpy="9.53145e-17 -4.66093e-24 0" />
+				<origin xyz="-5.55112e-17 0.0004 0.0189" rpy="9.53145e-17 -4.66093e-24 0" />
 				<geometry>
 					<mesh filename="package://so101_gazebo_demo/meshes/so101/moving_jaw_so101_v1.stl" />
@@ -414,14 +414,14 @@
 		<xacro:if value="$(arg gazebo_collision_primitives)">
 			<!-- Offline VHACD for the moving load-bearing fingertip only. -->
-			<xacro:fingertip_convex_collision piece="moving_jaw_contact_convex_000" directory="moving_jaw_contact" xyz="-5.55112e-17 -1.94746e-17 0.0189" rpy="9.53145e-17 -4.66093e-24 0" />
-			<xacro:fingertip_convex_collision piece="moving_jaw_contact_convex_001" directory="moving_jaw_contact" xyz="-5.55112e-17 -1.94746e-17 0.0189" rpy="9.53145e-17 -4.66093e-24 0" />
-			<xacro:fingertip_convex_collision piece="moving_jaw_contact_convex_002" directory="moving_jaw_contact" xyz="-5.55112e-17 -1.94746e-17 0.0189" rpy="9.53145e-17 -4.66093e-24 0" />
-			<xacro:fingertip_convex_collision piece="moving_jaw_contact_convex_003" directory="moving_jaw_contact" xyz="-5.55112e-17 -1.94746e-17 0.0189" rpy="9.53145e-17 -4.66093e-24 0" />
-			<xacro:fingertip_convex_collision piece="moving_jaw_contact_convex_004" directory="moving_jaw_contact" xyz="-5.55112e-17 -1.94746e-17 0.0189" rpy="9.53145e-17 -4.66093e-24 0" />
-			<xacro:fingertip_convex_collision piece="moving_jaw_contact_convex_005" directory="moving_jaw_contact" xyz="-5.55112e-17 -1.94746e-17 0.0189" rpy="9.53145e-17 -4.66093e-24 0" />
-			<xacro:fingertip_convex_collision piece="moving_jaw_contact_convex_006" directory="moving_jaw_contact" xyz="-5.55112e-17 -1.94746e-17 0.0189" rpy="9.53145e-17 -4.66093e-24 0" />
-			<xacro:fingertip_convex_collision piece="moving_jaw_contact_convex_007" directory="moving_jaw_contact" xyz="-5.55112e-17 -1.94746e-17 0.0189" rpy="9.53145e-17 -4.66093e-24 0" />
+			<xacro:fingertip_convex_collision piece="moving_jaw_contact_convex_000" directory="moving_jaw_contact" xyz="-5.55112e-17 0.0004 0.0189" rpy="9.53145e-17 -4.66093e-24 0" />
+			<xacro:fingertip_convex_collision piece="moving_jaw_contact_convex_001" directory="moving_jaw_contact" xyz="-5.55112e-17 0.0004 0.0189" rpy="9.53145e-17 -4.66093e-24 0" />
+			<xacro:fingertip_convex_collision piece="moving_jaw_contact_convex_002" directory="moving_jaw_contact" xyz="-5.55112e-17 0.0004 0.0189" rpy="9.53145e-17 -4.66093e-24 0" />
+			<xacro:fingertip_convex_collision piece="moving_jaw_contact_convex_003" directory="moving_jaw_contact" xyz="-5.55112e-17 0.0004 0.0189" rpy="9.53145e-17 -4.66093e-24 0" />
+			<xacro:fingertip_convex_collision piece="moving_jaw_contact_convex_004" directory="moving_jaw_contact" xyz="-5.55112e-17 0.0004 0.0189" rpy="9.53145e-17 -4.66093e-24 0" />
+			<xacro:fingertip_convex_collision piece="moving_jaw_contact_convex_005" directory="moving_jaw_contact" xyz="-5.55112e-17 0.0004 0.0189" rpy="9.53145e-17 -4.66093e-24 0" />
+			<xacro:fingertip_convex_collision piece="moving_jaw_contact_convex_006" directory="moving_jaw_contact" xyz="-5.55112e-17 0.0004 0.0189" rpy="9.53145e-17 -4.66093e-24 0" />
+			<xacro:fingertip_convex_collision piece="moving_jaw_contact_convex_007" directory="moving_jaw_contact" xyz="-5.55112e-17 0.0004 0.0189" rpy="9.53145e-17 -4.66093e-24 0" />
 		</xacro:if>
-		<xacro:configured_moving_fingertip_pad xyz="-5.55112e-17 -1.94746e-17 0.0189" rpy="9.53145e-17 -4.66093e-24 0" />
+		<xacro:configured_moving_fingertip_pad xyz="-5.55112e-17 0.0004 0.0189" rpy="9.53145e-17 -4.66093e-24 0" />
 	</link>
 	<!-- Joint from gripper to jaw -->
@@ -431,5 +431,5 @@
 		<child link="jaw" />
 		<axis xyz="0 0 1" />
-		<limit effort="10" velocity="10" lower="-0.059303612618397" upper="1.74533" />
+		<limit effort="10" velocity="10" lower="-0.059600220867817" upper="1.74533" />
 	</joint>
 	<transmission name="6_trans">

File: src/so101_gazebo_demo/urdf/so101_ros2_control.xacro (robot description, xacro)
@@ -48,5 +48,5 @@
         <joint name="6">
             <command_interface name="position">
-                <param name="min">-0.059303612618397</param>
+                <param name="min">-0.059600220867817</param>
                 <param name="max">1.74533</param>
             </command_interface>
