Commit message: refactor(so101): migrate C++ package runtime identity

File: src/so101_gazebo_demo_cpp/urdf/so101_base.xacro (robot description, xacro)
@@ -13,5 +13,5 @@
 			<origin xyz="${xyz}" rpy="${rpy}" />
 			<geometry>
-				<mesh filename="package://so101_gazebo_demo/meshes/so101/collision/${directory}/${piece}.stl" />
+				<mesh filename="package://so101_gazebo_demo_cpp/meshes/so101/collision/${directory}/${piece}.stl" />
 			</geometry>
 		</collision>
@@ -34,12 +34,12 @@
 			<xacro:property name="pads" value="${xacro.load_yaml('$(arg object_config)')['fingertip_pads']}" />
 			<xacro:if value="${pads['enabled']}">
-				<xacro:fingertip_pad_visual name="fixed_fingertip_pad" xyz="${xyz}" rpy="${rpy}" mesh="package://so101_gazebo_demo/meshes/so101/generated/fixed/fingertip_pad.stl" />
-				<xacro:fingertip_pad_collision name="fixed_fingertip_pad_collision_000" xyz="${xyz}" rpy="${rpy}" mesh="package://so101_gazebo_demo/meshes/so101/generated/fixed/fingertip_pad_collision_000.stl" />
-				<xacro:fingertip_pad_collision name="fixed_fingertip_pad_collision_001" xyz="${xyz}" rpy="${rpy}" mesh="package://so101_gazebo_demo/meshes/so101/generated/fixed/fingertip_pad_collision_001.stl" />
-				<xacro:fingertip_pad_collision name="fixed_fingertip_pad_collision_002" xyz="${xyz}" rpy="${rpy}" mesh="package://so101_gazebo_demo/meshes/so101/generated/fixed/fingertip_pad_collision_002.stl" />
-				<xacro:fingertip_pad_collision name="fixed_fingertip_pad_collision_003" xyz="${xyz}" rpy="${rpy}" mesh="package://so101_gazebo_demo/meshes/so101/generated/fixed/fingertip_pad_collision_003.stl" />
-				<xacro:fingertip_pad_collision name="fixed_fingertip_pad_collision_004" xyz="${xyz}" rpy="${rpy}" mesh="package://so101_gazebo_demo/meshes/so101/generated/fixed/fingertip_pad_collision_004.stl" />
-				<xacro:fingertip_pad_collision name="fixed_fingertip_pad_collision_005" xyz="${xyz}" rpy="${rpy}" mesh="package://so101_gazebo_demo/meshes/so101/generated/fixed/fingertip_pad_collision_005.stl" />
-				<xacro:fingertip_pad_collision name="fixed_fingertip_pad_collision_006" xyz="${xyz}" rpy="${rpy}" mesh="package://so101_gazebo_demo/meshes/so101/generated/fixed/fingertip_pad_collision_006.stl" />
+				<xacro:fingertip_pad_visual name="fixed_fingertip_pad" xyz="${xyz}" rpy="${rpy}" mesh="package://so101_gazebo_demo_cpp/meshes/so101/generated/fixed/fingertip_pad.stl" />
+				<xacro:fingertip_pad_collision name="fixed_fingertip_pad_collision_000" xyz="${xyz}" rpy="${rpy}" mesh="package://so101_gazebo_demo_cpp/meshes/so101/generated/fixed/fingertip_pad_collision_000.stl" />
+				<xacro:fingertip_pad_collision name="fixed_fingertip_pad_collision_001" xyz="${xyz}" rpy="${rpy}" mesh="package://so101_gazebo_demo_cpp/meshes/so101/generated/fixed/fingertip_pad_collision_001.stl" />
+				<xacro:fingertip_pad_collision name="fixed_fingertip_pad_collision_002" xyz="${xyz}" rpy="${rpy}" mesh="package://so101_gazebo_demo_cpp/meshes/so101/generated/fixed/fingertip_pad_collision_002.stl" />
+				<xacro:fingertip_pad_collision name="fixed_fingertip_pad_collision_003" xyz="${xyz}" rpy="${rpy}" mesh="package://so101_gazebo_demo_cpp/meshes/so101/generated/fixed/fingertip_pad_collision_003.stl" />
+				<xacro:fingertip_pad_collision name="fixed_fingertip_pad_collision_004" xyz="${xyz}" rpy="${rpy}" mesh="package://so101_gazebo_demo_cpp/meshes/so101/generated/fixed/fingertip_pad_collision_004.stl" />
+				<xacro:fingertip_pad_collision name="fixed_fingertip_pad_collision_005" xyz="${xyz}" rpy="${rpy}" mesh="package://so101_gazebo_demo_cpp/meshes/so101/generated/fixed/fingertip_pad_collision_005.stl" />
+				<xacro:fingertip_pad_collision name="fixed_fingertip_pad_collision_006" xyz="${xyz}" rpy="${rpy}" mesh="package://so101_gazebo_demo_cpp/meshes/so101/generated/fixed/fingertip_pad_collision_006.stl" />
 			</xacro:if>
 		</xacro:if>
@@ -49,11 +49,11 @@
 			<xacro:property name="pads" value="${xacro.load_yaml('$(arg object_config)')['fingertip_pads']}" />
 			<xacro:if value="${pads['enabled']}">
-				<xacro:fingertip_pad_visual name="moving_fingertip_pad" xyz="${xyz}" rpy="${rpy}" mesh="package://so101_gazebo_demo/meshes/so101/generated/moving/fingertip_pad.stl" />
-				<xacro:fingertip_pad_collision name="moving_fingertip_pad_collision_000" xyz="${xyz}" rpy="${rpy}" mesh="package://so101_gazebo_demo/meshes/so101/generated/moving/fingertip_pad_collision_000.stl" />
-				<xacro:fingertip_pad_collision name="moving_fingertip_pad_collision_001" xyz="${xyz}" rpy="${rpy}" mesh="package://so101_gazebo_demo/meshes/so101/generated/moving/fingertip_pad_collision_001.stl" />
-				<xacro:fingertip_pad_collision name="moving_fingertip_pad_collision_002" xyz="${xyz}" rpy="${rpy}" mesh="package://so101_gazebo_demo/meshes/so101/generated/moving/fingertip_pad_collision_002.stl" />
-				<xacro:fingertip_pad_collision name="moving_fingertip_pad_collision_003" xyz="${xyz}" rpy="${rpy}" mesh="package://so101_gazebo_demo/meshes/so101/generated/moving/fingertip_pad_collision_003.stl" />
-				<xacro:fingertip_pad_collision name="moving_fingertip_pad_collision_004" xyz="${xyz}" rpy="${rpy}" mesh="package://so101_gazebo_demo/meshes/so101/generated/moving/fingertip_pad_collision_004.stl" />
-				<xacro:fingertip_pad_collision name="moving_fingertip_pad_collision_005" xyz="${xyz}" rpy="${rpy}" mesh="package://so101_gazebo_demo/meshes/so101/generated/moving/fingertip_pad_collision_005.stl" />
+				<xacro:fingertip_pad_visual name="moving_fingertip_pad" xyz="${xyz}" rpy="${rpy}" mesh="package://so101_gazebo_demo_cpp/meshes/so101/generated/moving/fingertip_pad.stl" />
+				<xacro:fingertip_pad_collision name="moving_fingertip_pad_collision_000" xyz="${xyz}" rpy="${rpy}" mesh="package://so101_gazebo_demo_cpp/meshes/so101/generated/moving/fingertip_pad_collision_000.stl" />
+				<xacro:fingertip_pad_collision name="moving_fingertip_pad_collision_001" xyz="${xyz}" rpy="${rpy}" mesh="package://so101_gazebo_demo_cpp/meshes/so101/generated/moving/fingertip_pad_collision_001.stl" />
+				<xacro:fingertip_pad_collision name="moving_fingertip_pad_collision_002" xyz="${xyz}" rpy="${rpy}" mesh="package://so101_gazebo_demo_cpp/meshes/so101/generated/moving/fingertip_pad_collision_002.stl" />
+				<xacro:fingertip_pad_collision name="moving_fingertip_pad_collision_003" xyz="${xyz}" rpy="${rpy}" mesh="package://so101_gazebo_demo_cpp/meshes/so101/generated/moving/fingertip_pad_collision_003.stl" />
+				<xacro:fingertip_pad_collision name="moving_fingertip_pad_collision_004" xyz="${xyz}" rpy="${rpy}" mesh="package://so101_gazebo_demo_cpp/meshes/so101/generated/moving/fingertip_pad_collision_004.stl" />
+				<xacro:fingertip_pad_collision name="moving_fingertip_pad_collision_005" xyz="${xyz}" rpy="${rpy}" mesh="package://so101_gazebo_demo_cpp/meshes/so101/generated/moving/fingertip_pad_collision_005.stl" />
 			</xacro:if>
 		</xacro:if>
@@ -90,5 +90,5 @@
 			<geometry>
 				<mesh
-					filename="package://so101_gazebo_demo/meshes/so101/base_motor_holder_so101_v1.stl" />
+					filename="package://so101_gazebo_demo_cpp/meshes/so101/base_motor_holder_so101_v1.stl" />
 			</geometry>
 			<material name="3d_printed" />
@@ -98,5 +98,5 @@
 			<geometry>
 				<mesh
-					filename="package://so101_gazebo_demo/meshes/so101/base_motor_holder_so101_v1.stl" />
+					filename="package://so101_gazebo_demo_cpp/meshes/so101/base_motor_holder_so101_v1.stl" />
 			</geometry>
 		</collision>
@@ -105,5 +105,5 @@
 			<origin xyz="0.0207909 0.0221255 0.0300817" rpy="1.5708 -0 0" />
 			<geometry>
-				<mesh filename="package://so101_gazebo_demo/meshes/so101/base_so101_v2.stl" />
+				<mesh filename="package://so101_gazebo_demo_cpp/meshes/so101/base_so101_v2.stl" />
 			</geometry>
 			<material name="3d_printed" />
@@ -112,5 +112,5 @@
 			<origin xyz="0.0207909 0.0221255 0.0300817" rpy="1.5708 -0 0" />
 			<geometry>
-				<mesh filename="package://so101_gazebo_demo/meshes/so101/base_so101_v2.stl" />
+				<mesh filename="package://so101_gazebo_demo_cpp/meshes/so101/base_so101_v2.stl" />
 			</geometry>
 		</collision>
@@ -119,5 +119,5 @@
 			<origin xyz="0.0207909 -0.0105745 0.0761817" rpy="-2.20282e-15 2.77556e-17 -1.5708" />
 			<geometry>
-				<mesh filename="package://so101_gazebo_demo/meshes/so101/sts3215_03a_v1.stl" />
+				<mesh filename="package://so101_gazebo_demo_cpp/meshes/so101/sts3215_03a_v1.stl" />
 			</geometry>
 			<material name="sts3215" />
@@ -126,5 +126,5 @@
 			<origin xyz="0.0207909 -0.0105745 0.0761817" rpy="-2.20282e-15 2.77556e-17 -1.5708" />
 			<geometry>
-				<mesh filename="package://so101_gazebo_demo/meshes/so101/sts3215_03a_v1.stl" />
+				<mesh filename="package://so101_gazebo_demo_cpp/meshes/so101/sts3215_03a_v1.stl" />
 			</geometry>
 		</collision>
@@ -134,5 +134,5 @@
 			<geometry>
 				<mesh
-					filename="package://so101_gazebo_demo/meshes/so101/waveshare_mounting_plate_so101_v2.stl" />
+					filename="package://so101_gazebo_demo_cpp/meshes/so101/waveshare_mounting_plate_so101_v2.stl" />
 			</geometry>
 			<material name="3d_printed" />
@@ -142,5 +142,5 @@
 			<geometry>
 				<mesh
-					filename="package://so101_gazebo_demo/meshes/so101/waveshare_mounting_plate_so101_v2.stl" />
+					filename="package://so101_gazebo_demo_cpp/meshes/so101/waveshare_mounting_plate_so101_v2.stl" />
 			</geometry>
 		</collision>
@@ -158,5 +158,5 @@
 			<origin xyz="-0.0303992 0.000422241 -0.0417" rpy="1.5708 1.5708 0" />
 			<geometry>
-				<mesh filename="package://so101_gazebo_demo/meshes/so101/sts3215_03a_v1.stl" />
+				<mesh filename="package://so101_gazebo_demo_cpp/meshes/so101/sts3215_03a_v1.stl" />
 			</geometry>
 			<material name="sts3215" />
@@ -165,5 +165,5 @@
 			<origin xyz="-0.0303992 0.000422241 -0.0417" rpy="1.5708 1.5708 0" />
 			<geometry>
-				<mesh filename="package://so101_gazebo_demo/meshes/so101/sts3215_03a_v1.stl" />
+				<mesh filename="package://so101_gazebo_demo_cpp/meshes/so101/sts3215_03a_v1.stl" />
 			</geometry>
 		</collision>
@@ -173,5 +173,5 @@
 			<geometry>
 				<mesh
-					filename="package://so101_gazebo_demo/meshes/so101/motor_holder_so101_base_v1.stl" />
+					filename="package://so101_gazebo_demo_cpp/meshes/so101/motor_holder_so101_base_v1.stl" />
 			</geometry>
 			<material name="3d_printed" />
@@ -181,5 +181,5 @@
 			<geometry>
 				<mesh
-					filename="package://so101_gazebo_demo/meshes/so101/motor_holder_so101_base_v1.stl" />
+					filename="package://so101_gazebo_demo_cpp/meshes/so101/motor_holder_so101_base_v1.stl" />
 			</geometry>
 		</collision>
@@ -189,5 +189,5 @@
 			<geometry>
 				<mesh
-					filename="package://so101_gazebo_demo/meshes/so101/rotation_pitch_so101_v1.stl" />
+					filename="package://so101_gazebo_demo_cpp/meshes/so101/rotation_pitch_so101_v1.stl" />
 			</geometry>
 			<material name="3d_printed" />
@@ -197,5 +197,5 @@
 			<geometry>
 				<mesh
-					filename="package://so101_gazebo_demo/meshes/so101/rotation_pitch_so101_v1.stl" />
+					filename="package://so101_gazebo_demo_cpp/meshes/so101/rotation_pitch_so101_v1.stl" />
 			</geometry>
 		</collision>
@@ -213,5 +213,5 @@
 			<origin xyz="-0.11257 -0.0155 0.0187" rpy="-3.14159 -6.8695e-16 -1.5708" />
 			<geometry>
-				<mesh filename="package://so101_gazebo_demo/meshes/so101/sts3215_03a_v1.stl" />
+				<mesh filename="package://so101_gazebo_demo_cpp/meshes/so101/sts3215_03a_v1.stl" />
 			</geometry>
 			<material name="sts3215" />
@@ -220,5 +220,5 @@
 			<origin xyz="-0.11257 -0.0155 0.0187" rpy="-3.14159 -6.8695e-16 -1.5708" />
 			<geometry>
-				<mesh filename="package://so101_gazebo_demo/meshes/so101/sts3215_03a_v1.stl" />
+				<mesh filename="package://so101_gazebo_demo_cpp/meshes/so101/sts3215_03a_v1.stl" />
 			</geometry>
 		</collision>
@@ -227,5 +227,5 @@
 			<origin xyz="-0.065085 0.012 0.0182" rpy="3.14159 -9.35612e-32 0" />
 			<geometry>
-				<mesh filename="package://so101_gazebo_demo/meshes/so101/upper_arm_so101_v1.stl" />
+				<mesh filename="package://so101_gazebo_demo_cpp/meshes/so101/upper_arm_so101_v1.stl" />
 			</geometry>
 			<material name="3d_printed" />
@@ -234,5 +234,5 @@
 			<origin xyz="-0.065085 0.012 0.0182" rpy="3.14159 -9.35612e-32 0" />
 			<geometry>
-				<mesh filename="package://so101_gazebo_demo/meshes/so101/upper_arm_so101_v1.stl" />
+				<mesh filename="package://so101_gazebo_demo_cpp/meshes/so101/upper_arm_so101_v1.stl" />
 			</geometry>
 		</collision>
@@ -250,5 +250,5 @@
 			<origin xyz="-0.0648499 -0.032 0.0182" rpy="-3.14159 -0 3.9443e-31" />
 			<geometry>
-				<mesh filename="package://so101_gazebo_demo/meshes/so101/under_arm_so101_v1.stl" />
+				<mesh filename="package://so101_gazebo_demo_cpp/meshes/so101/under_arm_so101_v1.stl" />
 			</geometry>
 			<material name="3d_printed" />
@@ -257,5 +257,5 @@
 			<origin xyz="-0.0648499 -0.032 0.0182" rpy="-3.14159 -0 3.9443e-31" />
 			<geometry>
-				<mesh filename="package://so101_gazebo_demo/meshes/so101/under_arm_so101_v1.stl" />
+				<mesh filename="package://so101_gazebo_demo_cpp/meshes/so101/under_arm_so101_v1.stl" />
 			</geometry>
 		</collision>
@@ -265,5 +265,5 @@
 			<geometry>
 				<mesh
-					filename="package://so101_gazebo_demo/meshes/so101/motor_holder_so101_wrist_v1.stl" />
+					filename="package://so101_gazebo_demo_cpp/meshes/so101/motor_holder_so101_wrist_v1.stl" />
 			</geometry>
 			<material name="3d_printed" />
@@ -273,5 +273,5 @@
 			<geometry>
 				<mesh
-					filename="package://so101_gazebo_demo/meshes/so101/motor_holder_so101_wrist_v1.stl" />
+					filename="package://so101_gazebo_demo_cpp/meshes/so101/motor_holder_so101_wrist_v1.stl" />
 			</geometry>
 		</collision>
@@ -280,5 +280,5 @@
 			<origin xyz="-0.1224 0.0052 0.0187" rpy="-3.14159 -3.58047e-15 -3.14159" />
 			<geometry>
-				<mesh filename="package://so101_gazebo_demo/meshes/so101/sts3215_03a_v1.stl" />
+				<mesh filename="package://so101_gazebo_demo_cpp/meshes/so101/sts3215_03a_v1.stl" />
 			</geometry>
 			<material name="sts3215" />
@@ -287,5 +287,5 @@
 			<origin xyz="-0.1224 0.0052 0.0187" rpy="-3.14159 -3.58047e-15 -3.14159" />
 			<geometry>
-				<mesh filename="package://so101_gazebo_demo/meshes/so101/sts3215_03a_v1.stl" />
+				<mesh filename="package://so101_gazebo_demo_cpp/meshes/so101/sts3215_03a_v1.stl" />
 			</geometry>
 		</collision>
@@ -304,5 +304,5 @@
 			<geometry>
 				<mesh
-					filename="package://so101_gazebo_demo/meshes/so101/sts3215_03a_no_horn_v1.stl" />
+					filename="package://so101_gazebo_demo_cpp/meshes/so101/sts3215_03a_no_horn_v1.stl" />
 			</geometry>
 			<material name="sts3215" />
@@ -312,5 +312,5 @@
 			<geometry>
 				<mesh
-					filename="package://so101_gazebo_demo/meshes/so101/sts3215_03a_no_horn_v1.stl" />
+					filename="package://so101_gazebo_demo_cpp/meshes/so101/sts3215_03a_no_horn_v1.stl" />
 			</geometry>
 		</collision>
@@ -320,5 +320,5 @@
 			<geometry>
 				<mesh
-					filename="package://so101_gazebo_demo/meshes/so101/wrist_roll_pitch_so101_v2.stl" />
+					filename="package://so101_gazebo_demo_cpp/meshes/so101/wrist_roll_pitch_so101_v2.stl" />
 			</geometry>
 			<material name="3d_printed" />
@@ -328,5 +328,5 @@
 			<geometry>
 				<mesh
-					filename="package://so101_gazebo_demo/meshes/so101/wrist_roll_pitch_so101_v2.stl" />
+					filename="package://so101_gazebo_demo_cpp/meshes/so101/wrist_roll_pitch_so101_v2.stl" />
 			</geometry>
 		</collision>
@@ -344,5 +344,5 @@
 			<origin xyz="0.0077 0.0001 -0.0234" rpy="-1.5708 -5.55112e-17 -1.38213e-14" />
 			<geometry>
-				<mesh filename="package://so101_gazebo_demo/meshes/so101/sts3215_03a_v1.stl" />
+				<mesh filename="package://so101_gazebo_demo_cpp/meshes/so101/sts3215_03a_v1.stl" />
 			</geometry>
 			<material name="sts3215" />
@@ -352,5 +352,5 @@
 				<origin xyz="0.0077 0.0001 -0.0234" rpy="-1.5708 -5.55112e-17 -1.38213e-14" />
 				<geometry>
-					<mesh filename="package://so101_gazebo_demo/meshes/so101/sts3215_03a_v1.stl" />
+					<mesh filename="package://so101_gazebo_demo_cpp/meshes/so101/sts3215_03a_v1.stl" />
 				</geometry>
 			</collision>
@@ -362,5 +362,5 @@
 			<geometry>
 				<mesh
-					filename="package://so101_gazebo_demo/meshes/so101/wrist_roll_follower_so101_v1.stl" />
+					filename="package://so101_gazebo_demo_cpp/meshes/so101/wrist_roll_follower_so101_v1.stl" />
 			</geometry>
 			<material name="3d_printed" />
@@ -372,5 +372,5 @@
 				<geometry>
 					<mesh
-						filename="package://so101_gazebo_demo/meshes/so101/wrist_roll_follower_so101_v1.stl" />
+						filename="package://so101_gazebo_demo_cpp/meshes/so101/wrist_roll_follower_so101_v1.stl" />
 				</geometry>
 			</collision>
@@ -400,5 +400,5 @@
 			<origin xyz="-5.55112e-17 0.0004 0.0189" rpy="9.53145e-17 -4.66093e-24 0" />
 			<geometry>
-				<mesh filename="package://so101_gazebo_demo/meshes/so101/moving_jaw_so101_v1.stl" />
+				<mesh filename="package://so101_gazebo_demo_cpp/meshes/so101/moving_jaw_so101_v1.stl" />
 			</geometry>
 			<material name="3d_printed" />
@@ -408,5 +408,5 @@
 				<origin xyz="-5.55112e-17 0.0004 0.0189" rpy="9.53145e-17 -4.66093e-24 0" />
 				<geometry>
-					<mesh filename="package://so101_gazebo_demo/meshes/so101/moving_jaw_so101_v1.stl" />
+					<mesh filename="package://so101_gazebo_demo_cpp/meshes/so101/moving_jaw_so101_v1.stl" />
 				</geometry>
 			</collision>

File: src/so101_gazebo_demo_cpp/urdf/so101_gazebo.xacro (robot description, xacro)
@@ -4,5 +4,5 @@
     <gazebo>
         <plugin filename="gz_ros2_control-system" name="gz_ros2_control::GazeboSimROS2ControlPlugin">
-            <parameters>$(find so101_gazebo_demo)/config/so101_controllers.yaml</parameters>
+            <parameters>$(find so101_gazebo_demo_cpp)/config/so101_controllers.yaml</parameters>
         </plugin>
         <!--
