Commit message: fix(so101): close fusion provenance and asset ownership

File: src/so101_demo_py/assets/mujoco/so101.urdf (robot description, URDF)
Before this commit: robot so101, 9 links, 8 joints
Links:
- link base: geometry collision mesh filename=package://so101_demo_py/assets/common/visual/base_motor_hol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; collision mesh filename=package://so101_demo_py/assets/common/visual/base_so101_v2.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
- link gripper: geometry collision mesh filename=package://so101_demo_py/assets/mujoco/collision/fixed_finge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; collision mesh filename=package://so101_demo_py/assets/mujoco/collision/fixed_finge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
- link jaw: geometry collision mesh filename=package://so101_demo_py/assets/mujoco/collision/moving_fing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; collision mesh filename=package://so101_demo_py/assets/mujoco/collision/moving_fing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
- link lower_arm: geometry collision mesh filename=package://so101_demo_py/assets/common/visual/motor_holder_s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; collision mesh filename=package://so101_demo_py/assets/common/visual/sts3215_03a_v1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
- link shoulder: geometry collision mesh filename=package://so101_demo_py/assets/common/visual/motor_holder_s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; collision mesh filename=package://so101_demo_py/assets/common/visual/rotation_pitch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
- link upper_arm: geometry collision mesh filename=package://so101_demo_py/assets/common/visual/sts3215_03a_v1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; collision mesh filename=package://so101_demo_py/assets/common/visual/upper_arm_so10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
- link wrist: geometry collision mesh filename=package://so101_demo_py/assets/common/visual/sts3215_03a_no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; collision mesh filename=package://so101_demo_py/assets/common/visual/wrist_roll_pit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
