Commit message: fix: add world frame for SRDF virtual_joint in MuJoCo URDF
MuJoCo 版 URDF 缺少 world link，而系统 SRDF
(moveit_resources_panda_moveit_config) 定义了
virtual_joint parent_frame="world" child_link="panda_link0"，
导致 MoveIt PlanningSceneMonitor 持续报
'Missing virtual_joint' 且规划时无法定位机器人在 world 帧的位置。

与 Gazebo 版一致地添加 world link + 固定关节 world_to_panda。
区别在于 MuJoCo 把 panda_link0 直接置于世界原点（README 5.2），
所以该固定关节是零偏移单位变换，仅发布 TF world->panda_link0，
不改变 MuJoCo 物理坐标系。

File: src/panda_mujoco_demo/urdf/panda.mujoco.urdf.xacro (robot description, xacro)
@@ -4,4 +4,17 @@
         default="$(find panda_mujoco_demo)/config/initial_positions.yaml" />
     <xacro:arg name="headless" default="false" />
+    <!-- Provide the `world` frame the SRDF virtual_joint expects
+         (parent_frame="world", child_link="panda_link0"). Unlike the Gazebo
+         URDF, where world sits on the floor and panda_link0 is offset z=0.775
+         to the table top, the MuJoCo scene already centers panda_link0 at the
+         world origin (see README 5.2), so the fixed joint here is a zero-offset
+         identity transform. This only publishes TF world->panda_link0 for
+         MoveIt's PlanningSceneMonitor; it does not move the MuJoCo body. -->
+    <link name="world" />
+    <joint name="world_to_panda" type="fixed">
+        <parent link="world" />
+        <child link="panda_link0" />
+        <origin xyz="0 0 0" rpy="0 0 0" />
+    </joint>
     <!-- Import the kinematic/visual description (links + joints), verbatim from
          the Gazebo package so MoveIt and robot_state_publisher see identical
