Commit message: fix: tune friction and relax joint limits for MuJoCo grasp
scene.xml: table_top friction 10->1 (sliding mu=10 broke the contact solver, coke fell through the table to the floor); add friction to coke_body. panda.mjcf: friction on collision geoms, joint4 range -3.1416->-3.2. xacro: relax joint2/joint4 soft limits.

File: src/panda_mujoco_demo/urdf/panda.description.urdf.xacro (robot description, xacro)
@@ -77,6 +77,6 @@
     </link>
     <joint name="panda_joint2" type="revolute">
-        <safety_controller k_position="100.0" k_velocity="40.0" soft_lower_limit="-1.7628"
-            soft_upper_limit="1.7628" />
+        <safety_controller k_position="100.0" k_velocity="40.0" soft_lower_limit="-1.8326"
+            soft_upper_limit="1.8326" />
         <origin rpy="-1.57079632679 0 0" xyz="0 0 0" />
         <parent link="panda_link1" />
@@ -137,11 +137,11 @@
     </link>
     <joint name="panda_joint4" type="revolute">
-        <safety_controller k_position="100.0" k_velocity="40.0" soft_lower_limit="-3.0718"
-            soft_upper_limit="0.0175" />
+        <safety_controller k_position="100.0" k_velocity="40.0" soft_lower_limit="-3.2"
+            soft_upper_limit="0.0873" />
         <origin rpy="1.57079632679 0 0" xyz="0.0825 0 0" />
         <parent link="panda_link3" />
         <child link="panda_link4" />
         <axis xyz="0 0 1" />
-        <limit effort="87" lower="-3.1416" upper="0.0873" velocity="2.3925" />
+        <limit effort="87" lower="-3.2" upper="0.0873" velocity="2.3925" />
         <dynamics D="1" K="7000" damping="0.003" friction="0.0" mu_coulomb="0" mu_viscous="16" />
     </joint>
