Commit message: Aim ACT wrist camera at three scene cups

File: src/so101_demo_py/assets/mujoco/act/so101.urdf (robot description, URDF)
Before this commit: robot so101, 13 links, 12 joints
Joints:
- joint wrist_camera_optical_joint: origin xyz=0 0 0 rpy=3.141592653589793 0 0 -> xyz=0 0 0 rpy=2.6394826132462903 0.087724537669210845 -0.048065953798869021

Commit message: Calibrate ACT wrist camera for grasp candidate

File: src/so101_demo_py/assets/mujoco/act/so101.urdf (robot description, URDF)
Before this commit: robot so101, 13 links, 12 joints
Joints:
- joint wrist_camera_optical_joint: origin xyz=0 0 0 rpy=2.6394826132462903 0.087724537669210845 -0.048065953798869021 -> xyz=0 0 0 rpy=2.8353982087874967 0.18314198347413257 -0.078279728970571671

Commit message: WIP(head): checkpoint investigation and cross-host handoff

File: src/so101_demo_py/assets/mujoco/act/so101.urdf (robot description, URDF)
Before this commit: robot so101, 13 links, 12 joints
Links:
- link head_mount: geometry collision box size=0.036 0.024 0.024; visual box size=0.036 0.024 0.024
Joints:
- joint neck_yaw_joint: origin xyz=-0.06 0.06 0.24 rpy=0 0 0 -> xyz=-0.06 0.06 0.3892517831546664 rpy=0 0 0
