Commit message: Reconcile the Head merge: keep the local compiled model, drop the retired pick-place child stack, fix pytest-7 setup shadowing
- assets/mujoco/act/so101.xml and so101.urdf return to the local bytes. Head's neck height 0.389 m and camera
  housing geoms change the compiled model hash, which the user-activated contact policy (0ba8e07f...) and sixteen
  sealed profiles bind; adopting them needs a user decision (see CP-3527 follow-up).
- Remove the modify/delete files the merge resurrected from the Head line that only the retired pick-place
  child-port/search-boundary stack used, together with the seven tests that exercise only that stack.
  The Head modules that stay: ros_neck, broker_execution, controller_reservation_provision/client, pick_place_neck_sweep,
  pick_place_approach_goals, pick_place_readback (Head production and Head tests import them).
- test_b3_cleanup: ros_neck, broker_execution and controller_reservation_client are no longer on the deleted list and the
  C++ broker chain assertion allows the Head owned neck controller; command/ros broker, leased action client and the
  console script stay deleted.
- test_controller_reservation_provision: drop the standalone broker CLI test (the CLI is deleted by B3).
- so101_teleop.unified.controller_reservation_paths restored (imported by the Head reservation modules).
- test_act_head_original_router: rename the module-level setup() helper that pytest 7 ran as an xunit hook.

Co-Authored-By: Claude Sonnet 5.5 <noreply@anthropic.com>

File: src/so101_demo_py/assets/mujoco/act/so101.urdf (robot description, URDF)
Before this commit: robot so101, 13 links, 12 joints
Links:
- link head_mount: geometry collision box size=0.036 0.024 0.024; visual box size=0.036 0.024 0.024
Joints:
- joint neck_yaw_joint: origin xyz=-0.06 0.06 0.3892517831546664 rpy=0 0 0 -> xyz=-0.06 0.06 0.24 rpy=0 0 0
